File: hardware/electronics/driver-bldc-foc/driver-bldc-foc.kicad_pcb (KiCad board)
At the start: 2 copper layers, 19 parts, among them J1 VBUS, J2 GND, J3 USB_A, U2 STM32G473RETx, U3 AP1117-33

Commit message: link pcb footprint model
Parts:
- added C10: 100nF, Capacitor_SMD:C_0805_2012Metric, F.Cu at (296.7, 235.1)
- added C11: 100nF, Capacitor_SMD:C_0805_2012Metric, F.Cu at (296.7, 238.1)
- added C12: 10uF, Capacitor_SMD:C_0805_2012Metric, F.Cu at (296.7, 241.1)
- added C9: 1uF, Capacitor_SMD:C_0805_2012Metric, F.Cu at (296.7, 232.1)
- added J4: Motor_Phase_A, Connector_Wire:SolderWirePad_1x01_SMD_5x10mm, F.Cu at (297.8, 224.8)
- added J5: Motor_Phase_B, Connector_Wire:SolderWirePad_1x01_SMD_5x10mm, F.Cu at (304.4, 224.8)
- added J6: Motor_Phase_C, Connector_Wire:SolderWirePad_1x01_SMD_5x10mm, F.Cu at (311.0, 224.8)
- added L3: 1.5uH, Inductor_SMD:L_APV_ANR5040, F.Cu at (306.7, 233.9)
- added R3: 3k, Resistor_SMD:R_0805_2012Metric, F.Cu at (301.2, 232.1)
- added R4: 22k, Resistor_SMD:R_0805_2012Metric, F.Cu at (301.2, 235.0)
- added R5: 3k, Resistor_SMD:R_0805_2012Metric, F.Cu at (301.2, 238.0)
- added R6: 3k, Resistor_SMD:R_0805_2012Metric, F.Cu at (301.2, 240.9)
- added U1: TPS563240DDC, Package_TO_SOT_SMD:SOT-23-6, F.Cu at (305.9, 239.6)
- added U4: DRV8353RSRGZT, DRV8353RSRGZT:QFN50P700X700X100-49N, F.Cu at (321.5, 223.6)
