File: hardware/electronics/driver-bldc-foc/mcu.kicad_sch (KiCad schematic)
At the start: 23 parts, among them J7 Conn_01x04_Pin, U2 STM32G473RETx

Commit message: Update driver-bldc-foc schematics, PCB layout, and DRC reports
Parts:
- FB1, FB2: footprint Inductor_SMD:L_0201_0603Metric -> Inductor_SMD:L_0603_1608Metric_Pad1.05x0.95mm_HandSolder
Connections:
- net 3V3_IN: now also J7.1 (Pin_1), R27.2
- net 3V3_MCU: no longer J7.1 (Pin_1), R27.2
- no-connect marks 0 -> 13

Commit message: Complete PCB routing, fix net label connections, and export Gerber files for driver-bldc-foc
Parts:
- added J23, J24, J8: Conn_01x01_Pin, Connector_Wire:SolderWirePad_1x01_SMD_1x2mm, symbol Connector:Conn_01x01_Pin
Connections:
- net TIM2_CH1: now also J8.1 (Pin_1)
- net U1_RX: now also J23.1 (Pin_1)
- net U1_TX: now also J24.1 (Pin_1)
