File: hardware/electronics/driver-bldc-foc-v2/ThreePhaseBridgeandPower.kicad_sch (KiCad schematic)
At the start: 50 parts, among them Q1 BSC040N10NS5, Q2 BSC040N10NS5, Q3 BSC040N10NS5, Q4 BSC040N10NS5, Q5 BSC040N10NS5, Q6 BSC040N10NS5, U4 DRV8353RSRGZT

Commit message: update bridge schematic
Connections:
- net SPI_MISO: now also U4.29 (SDO); no longer R11.2, U4.30 (SDI)
- net SPI_MOSI: now also R11.2, U4.30 (SDI); no longer U4.29 (SDO)
Changed lines of the file:
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@@
 		)
 	)
-	(hierarchical_label "SPI_MISO"
+	(hierarchical_label "SPI_MOSI"
 		(shape input)
 		(at 66.04 86.36 180)
@@
 		)
 	)
-	(hierarchical_label "SPI_MOSI"
+	(hierarchical_label "SPI_MISO"
 		(shape input)
 		(at 81.28 88.9 180)
