File: hardware/electronics/driver-bldc-foc-v2/driver-bldc-foc-v2.kicad_pcb (KiCad board)
At the start: 4 copper layers, 80 x 60 mm, 117 parts, among them J1 Conn_01x01_Pin, J10 Conn_01x01_Pin, J11 Conn_01x01_Pin, J12 Conn_01x01_Pin, J13 Conn_01x01_Pin, J14 Conn_01x01_Pin, J15 Conn_01x01_Pin, J16 Conn_01x01_Pin, J17 Conn_01x01_Pin, J18 Conn_01x01_Pin, J19 Conn_01x01_Pin, J2 Conn_01x01_Pin, J20 Conn_01x01_Pin, J21 Conn_01x01_Pin, J22 Conn_01x01_Pin, J23 Conn_01x01_Pin, J24 Conn_01x01_Pin, J3 KH-TYPE-C-16P, J4 Motor_Phase_A, J5 Motor_Phase_B, J6 Motor_Phase_C, J7 Conn_01x04_Pin, J8 Conn_01x01_Pin, J9 Conn_01x01_Pin, Q1 BSC040N10NS5, Q2 BSC040N10NS5, Q3 BSC040N10NS5, Q4 BSC040N10NS5, Q5 BSC040N10NS5, Q6 BSC040N10NS5, U1 TPS563240DDC, U2 STM32G473RETx, U3 AP1117-33, U4 DRV8353RSRGZT, U5 TJA1051T-3, U6 XT30PW-M

Commit message: update board layout
Parts:
- added C46: 10uF, Capacitor_SMD:C_0805_2012Metric, F.Cu at (164.4, 154.9)
- added C47: 100nF, Capacitor_SMD:C_0805_2012Metric, F.Cu at (164.4, 157.9)
- added H1: MountingHole, MountingHole:MountingHole_3.2mm_M3_ISO7380_Pad_TopBottom, F.Cu at (174.0, 154.0)
- added H2: MountingHole, MountingHole:MountingHole_3.2mm_M3_ISO7380_Pad_TopBottom, F.Cu at (106.0, 106.0)
- added H3: MountingHole, MountingHole:MountingHole_3.2mm_M3_ISO7380_Pad_TopBottom, F.Cu at (106.0, 154.0)
- added H4: MountingHole, MountingHole:MountingHole_3.2mm_M3_ISO7380_Pad_TopBottom, F.Cu at (174.0, 106.0)
- moved R11 32.2 mm to (139.2, 139.7), turned to 0 degrees
- moved R10 3.84 mm to (173.2, 143.0)
- moved D4 3.68 mm to (173.2, 139.2)
- moved C19 0.15 mm to (164.4, 147.4)
- moved C20 0.15 mm to (164.4, 150.0)
Connections:
- R11 pad 2: /MCU/DRV_MISO -> /MCU/DRV_MOSI
- U4 pad 29: /MCU/DRV_MOSI -> /MCU/DRV_MISO
- U4 pad 30: /MCU/DRV_MISO -> /MCU/DRV_MOSI
Routing:
- net +3.3V: track 61.3 -> 38.8 mm, vias 63 -> 61
- net /MCU/DRV_MISO: track 39.2 -> 27.7 mm, vias 4 -> 2
- net /MCU/DRV_MOSI: track 35.9 -> 41.5 mm
- net /MCU/LED2: track 17.1 -> 20.0 mm
- net /MCU/3V3_MCU: track 109.7 -> 107.1 mm
- net GND: vias 177 -> 179
Other:
- outline, holes or cut-outs redrawn
- board text added: "V2"
