File: hardware/electronics/driver-bldc-foc-v2/driver-bldc-foc-v2.kicad_sch (KiCad schematic)
At the start: 41 parts, among them J1 Conn_01x01_Pin, J10 Conn_01x01_Pin, J11 Conn_01x01_Pin, J12 Conn_01x01_Pin, J13 Conn_01x01_Pin, J14 Conn_01x01_Pin, J15 Conn_01x01_Pin, J16 Conn_01x01_Pin, J17 Conn_01x01_Pin, J18 Conn_01x01_Pin, J19 Conn_01x01_Pin, J2 Conn_01x01_Pin, J20 Conn_01x01_Pin, J21 Conn_01x01_Pin, J22 Conn_01x01_Pin, J3 KH-TYPE-C-16P, J4 Motor_Phase_A, J5 Motor_Phase_B, J6 Motor_Phase_C, J9 Conn_01x01_Pin, U1 TPS563240DDC, U3 AP1117-33, U5 TJA1051T-3, U6 XT30PW-M

Commit message: update main schematic
Parts:
- added C46: 10uF, Capacitor_SMD:C_0805_2012Metric, symbol JLCPCB-Capacitors:0805,10uF
- added C47: 100nF, Capacitor_SMD:C_0805_2012Metric, symbol JLCPCB-Capacitors:0805,10uF
- added H1, H2, H3, H4: MountingHole, MountingHole:MountingHole_3.2mm_M3_ISO7380_Pad_TopBottom, symbol Mechanical:MountingHole
Connections:
- net 5V_BUCK: now also C46.1, C47.1
- net GND: now also C46.2, C47.2
